Commit message: home

File: urdf/リアルサイズ/main_robot.xacro (robot description, xacro)
@@ -4,11 +4,10 @@
   <xacro:include filename="$(find gazebo_sim)/urdf/wheel_macro.xacro"/>
   <xacro:include filename="$(find gazebo_sim)/urdf/caster_macro.xacro"/>
-  <xacro:wheel_macro prefix="left_wheel"  parent="base_link" xyz="0 0.13 0"/>
-  <xacro:wheel_macro prefix="right_wheel" parent="base_link" xyz="0 -0.13 0"/>
-  <xacro:ball_macro prefix="front_caster" parent="base_link" xyz="0.14 0 -0.06"/>
-  <xacro:ball_macro prefix="back_caster" parent="base_link" xyz="-0.14 0 -0.06"/>
-  <xacro:property name="x" value="0.4"/>
-  <xacro:property name="y" value="0.18"/>
-  <xacro:property name="z" value="0.1"/>
+  <xacro:wheel_macro prefix="left_wheel"  parent="base_link" xyz="-0.05 0.041 0"/>
+  <xacro:wheel_macro prefix="right_wheel" parent="base_link" xyz="-0.05 -0.041 0"/>
+  <xacro:ball_macro prefix="front_caster" parent="base_link" xyz="0.05 0 -0.03825"/>
+  <xacro:property name="x" value="0.14"/>
+  <xacro:property name="y" value="0.07"/>
+  <xacro:property name="z" value="0.05"/>
   <xacro:property name="mass" value="1.0"/>
   <link name="dummy"/>
@@ -16,5 +15,5 @@
     <parent link="dummy"/>
     <child link="base_link"/>
-    <origin xyz="0 0 0.1" rpy="0 0 0"/>
+    <origin xyz="0.05 0 0.0765" rpy="0 0 0"/>
   </joint>
   <link name="base_link">
@@ -29,7 +28,7 @@
       <origin xyz="0 0 0" rpy="0 0 0" />
       <geometry>
-        <box size="${x} ${y+0.02} ${z}" />
+        <box size="${x} ${y} ${z}" />
       </geometry>
-      <material name="gray" />
+      <material name="white" />
     </visual>
     <collision>
