Commit message: Update main_robot.xacro

File: urdf/main_robot.xacro (robot description, xacro)
@@ -4,19 +4,19 @@
   <xacro:include filename="$(find gazebo_sim)/urdf/wheel_macro.xacro"/>
   <xacro:include filename="$(find gazebo_sim)/urdf/caster_macro.xacro"/>
-  <xacro:wheel_macro prefix="left_wheel"  parent="base_link" xyz="0 0.13 0"/>
-  <xacro:wheel_macro prefix="right_wheel" parent="base_link" xyz="0 -0.13 0"/>
-  <xacro:ball_macro prefix="front_caster" parent="base_link" xyz="0.14 0 -0.06"/>
-  <xacro:ball_macro prefix="back_caster" parent="base_link" xyz="-0.14 0 -0.06"/>
+  <xacro:wheel_macro prefix="left_wheel"  parent="body_link" xyz="0 0.13 0"/>
+  <xacro:wheel_macro prefix="right_wheel" parent="body_link" xyz="0 -0.13 0"/>
+  <xacro:ball_macro prefix="front_caster" parent="body_link" xyz="0.14 0 -0.06"/>
+  <xacro:ball_macro prefix="back_caster" parent="body_link" xyz="-0.14 0 -0.06"/>
   <xacro:property name="x" value="0.4"/>
   <xacro:property name="y" value="0.18"/>
   <xacro:property name="z" value="0.1"/>
   <xacro:property name="mass" value="1.0"/>
-  <link name="dummy"/>
+  <link name="base_link"/>
   <joint name="base_joint" type="fixed">
-    <parent link="dummy"/>
-    <child link="base_link"/>
+    <parent link="base_link"/>
+    <child link="body_link"/>
     <origin xyz="0 0 0.1" rpy="0 0 0"/>
   </joint>
-  <link name="base_link">
+  <link name="body_link">
     <inertial>
      <origin xyz="0 0 0" rpy="0 0 0"/>
@@ -40,5 +40,5 @@
     </collision>
   </link>
-  <gazebo reference="base_link">
+  <gazebo reference="body_link">
    <material>Gazebo/Gray</material>
    <gravity>true</gravity>
