Commit message: home

File: urdf/caster_macro.xacro (robot description, xacro)
@@ -8,4 +8,9 @@
    </joint>
    <link name="${prefix}_link">
+    <inertial>
+      <origin xyz="0 0 0" rpy="0 0 0"/>
+      <mass value="0.2"/>
+      <inertia ixx="0.000128" ixy="0.0" ixz="0.0" iyy="0.000128" iyz="0.0" izz="0.000128"/>
+    </inertial>
     <visual>
       <origin xyz="0 0 0" rpy="0 0 0" />
@@ -13,5 +18,5 @@
         <sphere radius="0.04" />
       </geometry>
-      <material name="green" />
+      <material name="black" />
     </visual>
     <collision>
@@ -24,9 +29,7 @@
    </link>
    <gazebo reference="${prefix}_link">
-     <material>Gazebo/Green</material>
-     <mu1 value="0.5"/>
-     <mu2 value="0.5"/>
-     <kp value="50000"/>
-     <kd value="10"/>
+     <material>Gazebo/Black</material>
+     <mu1 value="0.0"/>
+     <mu2 value="0.0"/>
    </gazebo>
   </xacro:macro>

File: urdf/color.xacro (robot description, xacro)
@@ -13,3 +13,6 @@
    <color rgba="1.0 1.0 1.0 2.0"/>
   </material>
+  <material name="black">
+   <color rgba="0.0 0.0 0.0 2.0"/>
+  </material>
 </robot>

File: urdf/dtw_robot3.xacro (robot description, xacro)
@@ -13,4 +13,5 @@
       <child  link="${prefix}_link"/>
       <axis xyz="0 0 1" />
+      <dynamics damping="0.1"/>
     </joint>
     <transmission name="${prefix}_trans" type="SimpleTransmission">
@@ -43,8 +44,8 @@
     <gazebo reference="${prefix}_link">
       <material>Gazebo/Red</material>
-      <mu1 value="2.5" />
-      <mu2 value="2.5" />
-      <kp value="50000" />
-      <kd value="10" />
+      <mu1 value="1.0" />
+      <mu2 value="1.0" />
+      <kp value="10000000.0" />
+      <kd value="1.0" />
     </gazebo>
   </xacro:macro>
@@ -86,4 +87,9 @@
   </joint>
   <link name="ball_link">
+    <inertial>
+      <origin xyz="0 0 0" rpy="0 0 0"/>
+      <mass value="0.2"/>
+      <inertia ixx="0.000128" ixy="0.0" ixz="0.0" iyy="0.000128" iyz="0.0" izz="0.000128"/>
+    </inertial>
     <visual>
       <origin xyz="0 0 0" rpy="0 0 0" />
@@ -103,6 +109,6 @@
   <gazebo reference="ball_link">
     <material>Gazebo/Gray</material>
-    <mu1 value="0.5" />
-    <mu2 value="0.5" />
+    <mu1 value="0.0" />
+    <mu2 value="0.0" />
   </gazebo>
   <gazebo>

File: urdf/main_robot.xacro (robot description, xacro)
@@ -4,9 +4,8 @@
   <xacro:include filename="$(find gazebo_sim)/urdf/wheel_macro.xacro"/>
   <xacro:include filename="$(find gazebo_sim)/urdf/caster_macro.xacro"/>
-  <xacro:wheel_macro prefix="left_wheel"  parent="body_link" xyz="0 0.13 0"/>
-  <xacro:wheel_macro prefix="right_wheel" parent="body_link" xyz="0 -0.13 0"/>
-  <xacro:ball_macro prefix="front_caster" parent="body_link" xyz="0.14 0 -0.06"/>
-  <xacro:ball_macro prefix="back_caster" parent="body_link" xyz="-0.14 0 -0.06"/>
-  <xacro:property name="x" value="0.4"/>
+  <xacro:wheel_macro prefix="left_wheel"  parent="body_link" xyz="-0.1 0.13 0"/>
+  <xacro:wheel_macro prefix="right_wheel" parent="body_link" xyz="-0.1 -0.13 0"/>
+  <xacro:ball_macro prefix="front_caster" parent="body_link" xyz="0.1 0 -0.06"/>
+  <xacro:property name="x" value="0.3"/>
   <xacro:property name="y" value="0.18"/>
   <xacro:property name="z" value="0.1"/>
@@ -16,5 +15,5 @@
     <parent link="base_link"/>
     <child link="body_link"/>
-    <origin xyz="0 0 0.1" rpy="0 0 0"/>
+    <origin xyz="0.1 0 0.1" rpy="0 0 0"/>
   </joint>
   <link name="body_link">
@@ -31,5 +30,5 @@
         <box size="${x} ${y+0.02} ${z}" />
       </geometry>
-      <material name="gray" />
+      <material name="white" />
     </visual>
     <collision>
@@ -41,5 +40,5 @@
   </link>
   <gazebo reference="body_link">
-   <material>Gazebo/Gray</material>
+   <material>Gazebo/White</material>
    <gravity>true</gravity>
   </gazebo>

File: urdf/wheel_macro.xacro (robot description, xacro)
@@ -32,5 +32,5 @@
           <cylinder radius="${radius}" length="${length}" />
         </geometry>
-        <material name="red"/>
+        <material name="black"/>
       </visual>
       <collision>
@@ -41,7 +41,9 @@
     </link>
     <gazebo reference="${prefix}_link">
-     <material>Gazebo/Red</material>
-     <mu1 value="2.5"/>
-     <mu2 value="2.5"/>
+     <material>Gazebo/Black</material>
+     <mu1 value="1.0"/>
+     <mu2 value="1.0"/>
+     <kp value="10000000.0" />
+     <kd value="1.0" />
     </gazebo>
   </xacro:macro>

File: urdf/リアルサイズ/caster_macro.xacro (robot description, xacro)
@@ -10,8 +10,8 @@
     <inertial>
       <origin xyz="0 0 0" rpy="0 0 0"/>
-      <mass value="0.1"/>
-      <inertia ixx="${0.4*0.1*(0.03825**2)}" ixy="0.0" ixz="0.0"
-               iyy="${0.4*0.1*(0.03825**2)}" iyz="0.0"
-               izz="${0.4*0.1*(0.03825**2)}"/>
+      <mass value="0.04"/>
+      <inertia ixx="${0.4*0.04*(0.03825**2)}" ixy="0.0" ixz="0.0"
+               iyy="${0.4*0.04*(0.03825**2)}" iyz="0.0"
+               izz="${0.4*0.04*(0.03825**2)}"/>
     </inertial>
     <visual>
@@ -32,10 +32,6 @@
    <gazebo reference="${prefix}_link">
      <material>Gazebo/Green</material>
-     <mu1 value="1"/>
-     <mu2 value="1"/>
-     <!--
-     <kp value="50000"/>
-     <kd value="10"/>
-   -->
+     <mu1 value="0.0"/>
+     <mu2 value="0.0"/>
    </gazebo>
   </xacro:macro>

File: urdf/リアルサイズ/wheel_macro.xacro (robot description, xacro)
@@ -42,6 +42,8 @@
     <gazebo reference="${prefix}_link">
      <material>Gazebo/Red</material>
-     <mu1 value="2.5"/>
-     <mu2 value="2.5"/>
+     <mu1 value="1.0"/>
+     <mu2 value="1.0"/>
+     <kp value="10000000.0" />
+     <kd value="1.0" />
     </gazebo>
   </xacro:macro>

Commit message: school

File: urdf/caster_macro.xacro (robot description, xacro)
@@ -29,5 +29,5 @@
    </link>
    <gazebo reference="${prefix}_link">
-     <material>Gazebo/Black</material>
+     <material>Gazebo/Green</material>
      <mu1 value="0.0"/>
      <mu2 value="0.0"/>

File: urdf/wheel_macro.xacro (robot description, xacro)
@@ -32,5 +32,5 @@
           <cylinder radius="${radius}" length="${length}" />
         </geometry>
-        <material name="black"/>
+        <material name="red"/>
       </visual>
       <collision>
@@ -41,5 +41,5 @@
     </link>
     <gazebo reference="${prefix}_link">
-     <material>Gazebo/Black</material>
+     <material>Gazebo/Red</material>
      <mu1 value="1.0"/>
      <mu2 value="1.0"/>
